File: PCB/Rob/ROB.brd (EAGLE design)
At the start: 100 x 80 mm, 7 parts

Commit message: pcb files
Parts:
- removed J1: (no value), con-amp:1X6MTA
- added SV1: (no value), con-lstb:MA06-1
Connections:
- new net N$2: SV1.5
- net 5V: now also SV1.1, SV1.2; no longer J1.1, J1.2
- net GND: now also SV1.6; no longer J1.6
- net SCL: now also SV1.4; no longer J1.4
- net SDA: now also SV1.3; no longer J1.3
Routing:
- net GND: track 312.0 -> 308.7 mm
- net SCL: track 118.0 -> 120.9 mm
- net SDA: track 101.1 -> 103.1 mm
Changed lines of the file:
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@@
 <attribute name="VALUE" x="51.054" y="10.668" size="1.27" layer="27" ratio="10" rot="R90"/>
-</element>
-<element name="J1" library="con-amp" library_urn="urn:adsk.eagle:library:127" package="1X6MTA" package3d_urn="urn:adsk.eagle:package:8081593/1" value="" x="82.55" y="67.31" smashed="yes" rot="R180">
-<attribute name="NAME" x="86.8426" y="74.3712" size="1.778" layer="25" rot="R180"/>
-<attribute name="POPULARITY" value="1" x="57.15" y="110.49" size="1.778" layer="27" rot="R180" display="off"/>
-<attribute name="VALUE" x="93.9449" y="62.9592" size="1.27" layer="27" rot="R180"/>
 </element>
 <element name="J2" library="con-amp" library_urn="urn:adsk.eagle:library:127" package="10X04MTA" package3d_urn="urn:adsk.eagle:package:8081620/1" value="" x="13.97" y="15.24" smashed="yes" rot="R180">
@@
 <attribute name="VALUE" x="11.0569" y="69.2452" size="1.27" layer="27" rot="R180"/>
 </element>
+<element name="SV1" library="con-lstb" library_urn="urn:adsk.eagle:library:162" package="MA06-1" package3d_urn="urn:adsk.eagle:package:8340/1" value="" x="81.28" y="67.31" smashed="yes">
+<attribute name="MF" value="" x="81.28" y="67.31" size="1.778" layer="27" display="off"/>
+<attribute name="MPN" value="" x="81.28" y="67.31" size="1.778" layer="27" display="off"/>
+<attribute name="NAME" x="73.66" y="68.961" size="1.27" layer="25" ratio="10"/>
+<attribute name="OC_FARNELL" value="unknown" x="81.28" y="67.31" size="1.778" layer="27" display="off"/>
+<attribute name="OC_NEWARK" value="unknown" x="81.28" y="67.31" size="1.778" layer="27" display="off"/>
+<attribute name="POPULARITY" value="28" x="81.28" y="67.31" size="1.778" layer="27" display="off"/>
+<attribute name="VALUE" x="78.74" y="64.389" size="1.27" layer="27" ratio="10"/>
+</element>
 </elements>
 <signals>
 <signal name="SCL">
-<contactref element="J1" pad="4"/>
 <contactref element="BOARD1" pad="D22"/>
 <contactref element="J2" pad="3"/>
 <contactref element="J3" pad="3"/>
-<wire x1="84.5312" y1="67.31" x2="84.5312" y2="48.9712" width="1.27" layer="16"/>
 <wire x1="49.53" y1="34.29" x2="45.72" y2="30.48" width="1.27" layer="16"/>
 <wire x1="45.72" y1="30.48" x2="45.72" y2="25.4" width="1.27" layer="16"/>
-<wire x1="84.5312" y1="48.9712" x2="69.85" y2="34.29" width="1.27" layer="16"/>
-<wire x1="69.85" y1="34.29" x2="49.53" y2="34.29" width="1.27" layer="16"/>
 <wire x1="45.72" y1="25.4" x2="45.72" y2="24.13" width="1.27" layer="16"/>
 <wire x1="39.37" y1="21.59" x2="36.83" y2="19.05" width="1.27" layer="16"/>
@@
 <wire x1="15.24" y1="11.43" x2="15.24" y2="15.24" width="1.27" layer="16"/>
 <wire x1="36.83" y1="15.24" x2="36.83" y2="10.16" width="1.27" layer="16"/>
+<contactref element="SV1" pad="4"/>
+<wire x1="82.55" y1="67.31" x2="82.55" y2="40.64" width="1.27" layer="16"/>
+<wire x1="82.55" y1="40.64" x2="76.2" y2="34.29" width="1.27" layer="16"/>
+<wire x1="76.2" y1="34.29" x2="49.53" y2="34.29" width="1.27" layer="16"/>
 </signal>
 <signal name="SDA">
-<contactref element="J1" pad="3"/>
 <contactref element="BOARD1" pad="D21"/>
 <contactref element="J2" pad="4"/>
 <contactref element="J3" pad="4"/>
-<wire x1="80.5688" y1="67.31" x2="80.5688" y2="51.3588" width="1.27" layer="16"/>
 <wire x1="38.1" y1="31.75" x2="38.1" y2="25.4" width="1.27" layer="16"/>
-<wire x1="80.5688" y1="51.3588" x2="68.58" y2="39.37" width="1.27" layer="16"/>
-<wire x1="68.58" y1="39.37" x2="45.72" y2="39.37" width="1.27" layer="16"/>
 <wire x1="45.72" y1="39.37" x2="38.1" y2="31.75" width="1.27" layer="16"/>
 <wire x1="38.1" y1="25.4" x2="38.1" y2="24.13" width="1.27" layer="16"/>
@@
 <wire x1="38.1" y1="24.13" x2="34.29" y2="20.32" width="1.27" layer="16"/>
 <wire x1="17.78" y1="15.24" x2="34.29" y2="15.24" width="1.27" layer="16"/>
+<contactref element="SV1" pad="3"/>
+<wire x1="80.01" y1="67.31" x2="80.01" y2="46.99" width="1.27" layer="16"/>
+<wire x1="80.01" y1="46.99" x2="72.39" y2="39.37" width="1.27" layer="16"/>
+<wire x1="72.39" y1="39.37" x2="45.72" y2="39.37" width="1.27" layer="16"/>
 </signal>
 <signal name="GND">
 <contactref element="BOARD1" pad="GND"/>
 <contactref element="J2" pad="1"/>
-<contactref element="J1" pad="6"/>
 <contactref element="D1" pad="C"/>
 <contactref element="J3" pad="1"/>
@@
 <wire x1="50.8" y1="53.34" x2="46.99" y2="57.15" width="1.27" layer="16"/>
 <wire x1="39.37" y1="59.69" x2="39.37" y2="67.31" width="1.27" layer="16"/>
-<wire x1="92.456" y1="67.31" x2="92.456" y2="73.914" width="1.27" layer="16"/>
 <wire x1="39.37" y1="73.66" x2="39.37" y2="67.31" width="1.27" layer="16"/>
-<wire x1="92.456" y1="73.914" x2="88.9" y2="77.47" width="1.27" layer="16"/>
-<wire x1="88.9" y1="77.47" x2="43.18" y2="77.47" width="1.27" layer="16"/>
 <wire x1="43.18" y1="77.47" x2="39.37" y2="73.66" width="1.27" layer="16"/>
 <wire x1="41.91" y1="15.24" x2="41.91" y2="7.62" width="1.27" layer="16"/>
@@
 <wire x1="44.45" y1="3.81" x2="38.1" y2="3.81" width="1.27" layer="16"/>
 <wire x1="48.26" y1="7.62" x2="44.45" y2="3.81" width="1.27" layer="16"/>
-<wire x1="92.456" y1="67.31" x2="92.456" y2="27.686" width="1.27" layer="16"/>
-<wire x1="92.456" y1="27.686" x2="72.39" y2="7.62" width="1.27" layer="16"/>
-<wire x1="72.39" y1="7.62" x2="48.26" y2="7.62" width="1.27" layer="16"/>
+<contactref element="SV1" pad="6"/>
+<wire x1="87.63" y1="67.31" x2="87.63" y2="16.51" width="1.27" layer="16"/>
+<wire x1="87.63" y1="16.51" x2="78.74" y2="7.62" width="1.27" layer="16"/>
+<wire x1="78.74" y1="7.62" x2="48.26" y2="7.62" width="1.27" layer="16"/>
+<wire x1="87.63" y1="67.31" x2="87.63" y2="73.66" width="1.27" layer="16"/>
+<wire x1="87.63" y1="73.66" x2="83.82" y2="77.47" width="1.27" layer="16"/>
+<wire x1="83.82" y1="77.47" x2="43.18" y2="77.47" width="1.27" layer="16"/>
 </signal>
 <signal name="5V">
 <contactref element="BOARD1" pad="VIN"/>
 <contactref element="J2" pad="2"/>
-<contactref element="J1" pad="2"/>
-<contactref element="J1" pad="1"/>
 <contactref element="J3" pad="2"/>
 <contactref element="J4" pad="4"/>
@@
 <wire x1="12.7" y1="50.8" x2="12.7" y2="48.26" width="1.27" layer="16"/>
 <wire x1="12.7" y1="48.26" x2="16.51" y2="44.45" width="1.27" layer="16"/>
-<wire x1="72.644" y1="52.324" x2="72.644" y2="67.31" width="1.27" layer="16"/>
 <wire x1="16.51" y1="44.45" x2="64.77" y2="44.45" width="1.27" layer="16"/>
-<wire x1="64.77" y1="44.45" x2="72.644" y2="52.324" width="1.27" layer="16"/>
-<wire x1="72.644" y1="67.31" x2="76.6064" y2="67.31" width="1.27" layer="16"/>
 <wire x1="10.16" y1="38.1" x2="16.51" y2="44.45" width="1.27" layer="16"/>
 <wire x1="39.37" y1="15.24" x2="39.37" y2="8.89" width="1.27" layer="16"/>
@@
 <wire x1="12.7" y1="19.05" x2="10.16" y2="21.59" width="1.27" layer="16"/>
 <wire x1="10.16" y1="21.59" x2="10.16" y2="38.1" width="1.27" layer="16"/>
+<contactref element="SV1" pad="2"/>
+<contactref element="SV1" pad="1"/>
+<wire x1="74.93" y1="54.61" x2="74.93" y2="67.31" width="1.27" layer="16"/>
+<wire x1="64.77" y1="44.45" x2="74.93" y2="54.61" width="1.27" layer="16"/>
+<wire x1="74.93" y1="67.31" x2="77.47" y2="67.31" width="1.27" layer="16"/>
 </signal>
 <signal name="LED">
@@
 <wire x1="34.29" y1="59.69" x2="27.94" y2="53.34" width="1.27" layer="16"/>
 </signal>
+<signal name="N$2">
+<contactref element="SV1" pad="5"/>
+</signal>
 </signals>
