File: PCB/Rob/ROB.sch (EAGLE design)
At the start: 7 parts

Commit message: pcb files
Parts:
- removed J1: (no value), con-amp:MTA06-156
- added SV1: (no value), con-lstb:MA06-1
Connections:
- new net N$2: SV1.5
- net 5V: now also SV1.1, SV1.2; no longer J1.1, J1.2
- net GND: now also SV1.6; no longer J1.6
- net SCL: now also SV1.4; no longer J1.4
- net SDA: now also SV1.3; no longer J1.3
Changed lines of the file:
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@@
 <parts>
 <part name="BOARD1" library="ESP32-DEVKITV1" deviceset="ESP32DEVKITV1" device=""/>
-<part name="J1" library="con-amp" library_urn="urn:adsk.eagle:library:127" deviceset="MTA06-156" device="" package3d_urn="urn:adsk.eagle:package:8081593/1"/>
 <part name="J2" library="con-amp" library_urn="urn:adsk.eagle:library:127" deviceset="MTA04-100" device="" package3d_urn="urn:adsk.eagle:package:8081620/1"/>
 <part name="D1" library="diode" library_urn="urn:adsk.eagle:library:210" deviceset="1N4004" device="" package3d_urn="urn:adsk.eagle:package:43336/1"/>
@@
 <part name="J4" library="con-amp" library_urn="urn:adsk.eagle:library:127" deviceset="MTA05-100" device="" package3d_urn="urn:adsk.eagle:package:8081622/1"/>
 <part name="J5" library="con-amp" library_urn="urn:adsk.eagle:library:127" deviceset="MTA02-156" device="" package3d_urn="urn:adsk.eagle:package:8081562/1"/>
+<part name="SV1" library="con-lstb" library_urn="urn:adsk.eagle:library:162" deviceset="MA06-1" device="" package3d_urn="urn:adsk.eagle:package:8340/1"/>
 </parts>
 <sheets>
@@
 <attribute name="NAME" x="51.435" y="73.025" size="1.27" layer="95"/>
 </instance>
-<instance part="J1" gate="G$1" x="139.7" y="50.8" smashed="yes" rot="R90">
-<attribute name="NAME" x="139.7" y="66.04" size="1.778" layer="95" rot="R90"/>
-<attribute name="VALUE" x="143.51" y="66.04" size="1.778" layer="96" rot="R90"/>
-</instance>
 <instance part="J2" gate="G$1" x="142.24" y="40.64" smashed="yes">
 <attribute name="NAME" x="149.86" y="40.64" size="1.778" layer="95"/>
@@
 <attribute name="NAME" x="-10.16" y="17.78" size="1.778" layer="95"/>
 <attribute name="VALUE" x="-10.16" y="13.97" size="1.778" layer="96"/>
+</instance>
+<instance part="SV1" gate="1" x="116.84" y="5.08" smashed="yes">
+<attribute name="VALUE" x="115.57" y="-7.62" size="1.778" layer="96"/>
+<attribute name="NAME" x="115.57" y="13.462" size="1.778" layer="95"/>
 </instance>
 </instances>
@@
 <net name="SCL" class="0">
 <segment>
-<pinref part="J1" gate="G$1" pin="4"/>
-<wire x1="142.24" y1="58.42" x2="154.94" y2="58.42" width="0.1524" layer="91"/>
-<label x="160.02" y="58.42" size="1.778" layer="95"/>
-</segment>
-<segment>
 <pinref part="BOARD1" gate="G$1" pin="D22"/>
 <wire x1="86.36" y1="58.42" x2="99.06" y2="58.42" width="0.1524" layer="91"/>
@@
 <label x="165.1" y="17.78" size="1.778" layer="95"/>
 </segment>
+<segment>
+<pinref part="SV1" gate="1" pin="4"/>
+<wire x1="124.46" y1="5.08" x2="134.62" y2="5.08" width="0.1524" layer="91"/>
+<label x="139.7" y="5.08" size="1.778" layer="95"/>
+</segment>
 </net>
 <net name="SDA" class="0">
-<segment>
-<pinref part="J1" gate="G$1" pin="3"/>
-<wire x1="142.24" y1="55.88" x2="154.94" y2="55.88" width="0.1524" layer="91"/>
-<label x="160.02" y="55.88" size="1.778" layer="95"/>
-</segment>
 <segment>
 <pinref part="BOARD1" gate="G$1" pin="D21"/>
@@
 <wire x1="167.64" y1="38.1" x2="167.64" y2="27.94" width="0.1524" layer="91"/>
 <label x="167.64" y="15.24" size="1.778" layer="95"/>
+</segment>
+<segment>
+<pinref part="SV1" gate="1" pin="3"/>
+<wire x1="124.46" y1="2.54" x2="134.62" y2="2.54" width="0.1524" layer="91"/>
+<label x="139.7" y="2.54" size="1.778" layer="95"/>
 </segment>
 </net>
@@
 </segment>
 <segment>
-<pinref part="J1" gate="G$1" pin="6"/>
-<wire x1="142.24" y1="63.5" x2="154.94" y2="63.5" width="0.1524" layer="91"/>
-<label x="160.02" y="63.5" size="1.778" layer="95"/>
-</segment>
-<segment>
 <pinref part="D1" gate="1" pin="C"/>
 <wire x1="144.78" y1="76.2" x2="160.02" y2="76.2" width="0.1524" layer="91"/>
@@
 <label x="-12.7" y="0" size="1.778" layer="95"/>
 </segment>
+<segment>
+<pinref part="SV1" gate="1" pin="6"/>
+<wire x1="124.46" y1="10.16" x2="134.62" y2="10.16" width="0.1524" layer="91"/>
+<label x="139.7" y="10.16" size="1.778" layer="95"/>
+</segment>
 </net>
 <net name="5V" class="0">
@@
 </segment>
 <segment>
-<pinref part="J1" gate="G$1" pin="2"/>
-<wire x1="142.24" y1="53.34" x2="154.94" y2="53.34" width="0.1524" layer="91"/>
-<label x="160.02" y="53.34" size="1.778" layer="95"/>
-</segment>
-<segment>
-<pinref part="J1" gate="G$1" pin="1"/>
-<wire x1="142.24" y1="50.8" x2="154.94" y2="50.8" width="0.1524" layer="91"/>
-<label x="160.02" y="50.8" size="1.778" layer="95"/>
-</segment>
-<segment>
 <pinref part="J3" gate="G$1" pin="2"/>
 <wire x1="162.56" y1="38.1" x2="162.56" y2="27.94" width="0.1524" layer="91"/>
@@
 <wire x1="-15.24" y1="15.24" x2="-15.24" y2="7.62" width="0.1524" layer="91"/>
 <label x="-15.24" y="-5.08" size="1.778" layer="95"/>
+</segment>
+<segment>
+<pinref part="SV1" gate="1" pin="2"/>
+<wire x1="124.46" y1="0" x2="134.62" y2="0" width="0.1524" layer="91"/>
+<label x="139.7" y="0" size="1.778" layer="95"/>
+</segment>
+<segment>
+<pinref part="SV1" gate="1" pin="1"/>
+<wire x1="124.46" y1="-2.54" x2="134.62" y2="-2.54" width="0.1524" layer="91"/>
+<label x="139.7" y="-2.54" size="1.778" layer="95"/>
 </segment>
 </net>
@@
 </segment>
 </net>
+<net name="N$2" class="0">
+<segment>
+<pinref part="SV1" gate="1" pin="5"/>
+<wire x1="124.46" y1="7.62" x2="134.62" y2="7.62" width="0.1524" layer="91"/>
+</segment>
+</net>
