File: PCB/ROB v2/ROB v2.brd (EAGLE design)
At the start: 100 x 80 mm, 14 parts, among them IC1 1182-A4988, IC2 1182-A4988, IC3 1182-A4988, J1 455-1750-1-ND, J2 455-1750-1-ND

Commit message: updated schematics and board
Parts:
- removed J1, J2: 455-1750-1-ND, SparkFun-Connectors:1X03
- added D1: (no value), BeagleBone_Blue_R3:DIODE-1N4001-KIT
- added SERVO1, SERVO2: 455-1750-1-ND, SparkFun-Connectors:1X03
- moved C1 171.4 mm to (95.4, 32.0), turned to 270 degrees
- moved J5 136.3 mm to (93.0, 17.3), turned to 270 degrees
- moved IC2 124.3 mm to (80.9, 13.5)
- moved FAN 120.8 mm to (95.1, 52.1)
- moved J6 117.0 mm to (67.0, 34.7), turned to 270 degrees
- moved 5VPOWERSUPPLY 117.0 mm to (50.1, 51.2), turned to 270 degrees
- moved J4 116.5 mm to (92.0, 46.9), turned to 270 degrees
- moved 12V-POWER 113.9 mm to (95.5, 59.1)
- moved IC3 111.6 mm to (55.4, 30.5)
- moved IC1 102.2 mm to (80.4, 43.5)
- moved BOARD1 91.9 mm to (35.9, 10.1), turned to 90 degrees
- moved J7 89.9 mm to (27.9, 35.7), turned to 90 degrees
Connections:
- new net LED: BOARD1.D15, D1.A
- net 5V: now also SERVO1.2, SERVO2.2; no longer J1.2, J2.2
- net GND: now also BOARD1.GND@1, D1.C, SERVO1.3, SERVO2.3; no longer BOARD1.GND, J1.3, J2.3
- net SIG1: now also SERVO2.1; no longer J2.1
- net SIG2: now also SERVO1.1; no longer J1.1
Routing:
- net GND: track 0.00 -> 294.8 mm
- net 5V: track 0.00 -> 233.6 mm
- net DIR1: track 0.00 -> 144.5 mm
- net 12V: track 0.00 -> 121.5 mm
- net SIG2: track 0.00 -> 98.7 mm
- net DIR2: track 0.00 -> 84.6 mm
- net STEP2: track 0.00 -> 81.7 mm
- net SIG1: track 0.00 -> 70.7 mm
- net DIR3: track 0.00 -> 63.0 mm
- net STEP1: track 0.00 -> 52.1 mm
- net STEP3: track 0.00 -> 13.6 mm
- net LED: track 0.00 -> 11.4 mm
- net SCL: track 0.00 -> 11.3 mm
- net SDA: track 0.00 -> 8.25 mm
- net 1B2: track 0.00 -> 5.81 mm
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Other:
- board size 100 x 80 mm -> 100 x 62 mm
- board text added: "ROB ver 2.0"
