File: PCB/ROB v2/ROB v2.sch (EAGLE design)
At the start: 14 parts, among them IC1 1182-A4988, IC2 1182-A4988, IC3 1182-A4988, J1 455-1750-1-ND, J2 455-1750-1-ND

Commit message: updated schematics and board
Parts:
- added D1: (no value), BeagleBone_Blue_R3:DIODE
- renumbered J1 to SERVO1, J2 to SERVO2
Connections:
- new net LED: BOARD1.D15, D1.A
- net GND: now also BOARD1.GND@1, D1.C; no longer BOARD1.GND
Changed lines of the file:
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@@
 <part name="J7" library="SparkFun-Connectors" library_urn="urn:adsk.eagle:library:513" deviceset="CONN_04" device="LOCK" package3d_urn="urn:adsk.eagle:package:38089/2"/>
 <part name="C1" library="BeagleBone_Black_Wireless" library_urn="urn:adsk.eagle:library:6644236" deviceset="C-US" device="050-075X075" package3d_urn="urn:adsk.eagle:package:8118548/1"/>
-<part name="J1" library="SparkFun-Connectors" library_urn="urn:adsk.eagle:library:513" deviceset="CONN_03" device="" package3d_urn="urn:adsk.eagle:package:38063/2" value="455-1750-1-ND"/>
-<part name="J2" library="SparkFun-Connectors" library_urn="urn:adsk.eagle:library:513" deviceset="CONN_03" device="" package3d_urn="urn:adsk.eagle:package:38063/2" value="455-1750-1-ND"/>
+<part name="SERVO1" library="SparkFun-Connectors" library_urn="urn:adsk.eagle:library:513" deviceset="CONN_03" device="" package3d_urn="urn:adsk.eagle:package:38063/2" value="455-1750-1-ND"/>
+<part name="SERVO2" library="SparkFun-Connectors" library_urn="urn:adsk.eagle:library:513" deviceset="CONN_03" device="" package3d_urn="urn:adsk.eagle:package:38063/2" value="455-1750-1-ND"/>
+<part name="D1" library="BeagleBone_Blue_R3" library_urn="urn:adsk.eagle:library:5828899" deviceset="DIODE" device="" package3d_urn="urn:adsk.eagle:package:5829545/1"/>
 </parts>
 <sheets>
@@
 <attribute name="VALUE" x="51.816" y="87.249" size="1.778" layer="96"/>
 </instance>
-<instance part="J1" gate="J1" x="10.16" y="15.24" smashed="yes">
+<instance part="SERVO1" gate="J1" x="10.16" y="15.24" smashed="yes">
 <attribute name="VALUE" x="7.62" y="7.874" size="1.778" layer="96" font="vector"/>
 <attribute name="NAME" x="7.62" y="20.828" size="1.778" layer="95" font="vector"/>
 </instance>
-<instance part="J2" gate="J1" x="10.16" y="0" smashed="yes">
+<instance part="SERVO2" gate="J1" x="10.16" y="0" smashed="yes">
 <attribute name="VALUE" x="7.62" y="-7.366" size="1.778" layer="96" font="vector"/>
 <attribute name="NAME" x="7.62" y="5.588" size="1.778" layer="95" font="vector"/>
+</instance>
+<instance part="D1" gate="G$1" x="114.3" y="-10.16" smashed="yes">
+<attribute name="NAME" x="116.84" y="-9.6774" size="1.778" layer="95"/>
+<attribute name="VALUE" x="116.84" y="-12.4714" size="1.778" layer="96"/>
 </instance>
 </instances>
@@
 </segment>
 <segment>
-<pinref part="J2" gate="J1" pin="2"/>
+<pinref part="SERVO2" gate="J1" pin="2"/>
 <wire x1="17.78" y1="0" x2="33.02" y2="0" width="0.1524" layer="91"/>
 <label x="38.1" y="0" size="1.778" layer="95"/>
 </segment>
 <segment>
-<pinref part="J1" gate="J1" pin="2"/>
+<pinref part="SERVO1" gate="J1" pin="2"/>
 <wire x1="17.78" y1="15.24" x2="33.02" y2="15.24" width="0.1524" layer="91"/>
 <label x="38.1" y="15.24" size="1.778" layer="95"/>
@@
 </net>
 <net name="GND" class="0">
-<segment>
-<pinref part="BOARD1" gate="G$1" pin="GND"/>
-<wire x1="71.12" y1="35.56" x2="60.96" y2="35.56" width="0.1524" layer="91"/>
-<label x="48.26" y="35.56" size="1.778" layer="95"/>
-</segment>
 <segment>
 <pinref part="FAN" gate="J1" pin="2"/>
@@
 </segment>
 <segment>
-<pinref part="J2" gate="J1" pin="3"/>
+<pinref part="SERVO2" gate="J1" pin="3"/>
 <wire x1="17.78" y1="2.54" x2="33.02" y2="2.54" width="0.1524" layer="91"/>
 <wire x1="33.02" y1="2.54" x2="33.02" y2="5.08" width="0.1524" layer="91"/>
@@
 </segment>
 <segment>
-<pinref part="J1" gate="J1" pin="3"/>
+<pinref part="SERVO1" gate="J1" pin="3"/>
 <wire x1="17.78" y1="17.78" x2="33.02" y2="17.78" width="0.1524" layer="91"/>
 <label x="38.1" y="17.78" size="1.778" layer="95"/>
+</segment>
+<segment>
+<pinref part="D1" gate="G$1" pin="C"/>
+<wire x1="116.84" y1="-10.16" x2="124.46" y2="-10.16" width="0.1524" layer="91"/>
+<label x="129.54" y="-10.16" size="1.778" layer="95"/>
+</segment>
+<segment>
+<pinref part="BOARD1" gate="G$1" pin="GND@1"/>
+<wire x1="111.76" y1="35.56" x2="121.92" y2="35.56" width="0.1524" layer="91"/>
+<label x="124.46" y="35.56" size="1.778" layer="95"/>
 </segment>
 </net>
@@
 <net name="SIG2" class="0">
 <segment>
-<pinref part="J1" gate="J1" pin="1"/>
+<pinref part="SERVO1" gate="J1" pin="1"/>
 <wire x1="17.78" y1="12.7" x2="30.48" y2="12.7" width="0.1524" layer="91"/>
 <label x="38.1" y="12.7" size="1.778" layer="95"/>
@@
 <net name="SIG1" class="0">
 <segment>
-<pinref part="J2" gate="J1" pin="1"/>
+<pinref part="SERVO2" gate="J1" pin="1"/>
 <wire x1="17.78" y1="-2.54" x2="33.02" y2="-2.54" width="0.1524" layer="91"/>
 <label x="38.1" y="-2.54" size="1.778" layer="95"/>
@@
 </segment>
 </net>
+<net name="LED" class="0">
+<segment>
+<pinref part="BOARD1" gate="G$1" pin="D15"/>
+<wire x1="111.76" y1="38.1" x2="119.38" y2="38.1" width="0.1524" layer="91"/>
+<label x="124.46" y="38.1" size="1.778" layer="95"/>
+</segment>
+<segment>
+<pinref part="D1" gate="G$1" pin="A"/>
+<wire x1="111.76" y1="-10.16" x2="104.14" y2="-10.16" width="0.1524" layer="91"/>
+<label x="93.98" y="-10.16" size="1.778" layer="95"/>
+</segment>
+</net>
